Commit message: Update xacro files to make them displayable

File: robotiq_description/urdf/robotiq_140_gripper.xacro (robot description, xacro)
@@ -1,5 +1,39 @@
-<?xml version="1.0"?>
-<robot name="robotiq_140_gripper" xmlns:xacro="http://ros.org/wiki/xacro">
+<?xml version="1.0" ?>
+<robot name="robotiq_140_gripper" xmlns:xacro="http://www.ros.org/wiki/xacro">
   <xacro:include filename="$(find robotiq_description)/urdf/robotiq_140_gripper.urdf.xacro" />
-  <xacro:robotiq_140_gripper prefix=""/>
+  <gazebo>
+    <plugin name="gazebo_ros_control" filename="libgazebo_ros_control.so">
+      <robotNamespace>/</robotNamespace>
+    </plugin>
+  </gazebo>
+  <link name="world"/>
+  <joint name="world_fixed" type="fixed">
+    <origin xyz="0 0 0" rpy="0 0 0"/>
+    <parent link="world"/>
+    <child link="gripper_root_link"/>
+  </joint>
+  <link name="gripper_root_link">
+    <visual>
+      <origin xyz="0 0 0.5" rpy="0 0 0"/>
+      <geometry>
+        <box size="0.1 0.1 1.0"/>
+      </geometry>
+    </visual>
+    <collision>
+      <origin xyz="0 0 0.5" rpy="0 0 0"/>
+      <geometry>
+        <box size="0.1 0.1 1.0"/>
+      </geometry>
+    </collision>
+    <inertial>
+      <mass value="1e2" />
+      <origin xyz="0.0 0.0 0.0" />
+      <inertia ixx = "0.000001" ixy = "0.000000" ixz = "0.000000"
+           iyx = "0.000000" iyy = "0.000001" iyz = "0.000000"
+           izx = "0.000000" izy = "0.000000" izz = "0.000001" />
+    </inertial>
+  </link>
+  <xacro:robotiq_140_gripper prefix="" parent="gripper_root_link" >
+    <origin xyz="0.05 0 0.140" rpy="0 0 0"/>
+  </xacro:robotiq_140_gripper>
 </robot>

File: robotiq_description/urdf/robotiq_85_gripper.xacro (robot description, xacro)
@@ -1,5 +1,5 @@
 <?xml version="1.0" ?>
 <robot name="robotiq_85_gripper" xmlns:xacro="http://www.ros.org/wiki/xacro">
-  <xacro:include filename="$(find robotiq_description)/urdf/robotiq_85_gripper_cb.urdf.xacro" />
+  <xacro:include filename="$(find robotiq_description)/urdf/robotiq_85_gripper.urdf.xacro" />
   <gazebo>
     <plugin name="gazebo_ros_control" filename="libgazebo_ros_control.so">
