Commit message: Clean up and kinetic compliant changes

File: robotiq_description/urdf/robotiq_85_gripper_sim_base.urdf.xacro (robot description, xacro)
@@ -1,26 +1,26 @@
 <?xml version="1.0"?>
-<robot name="robotiq_85_gripper_sim_base" xmlns:xacro="http://ros.org/wiki/xacro">
-    <xacro:macro name="robotiq_85_gripper_sim_base" params="prefix">
-        <link name="${prefix}gripper_root_link">
-            <visual>
-                <origin xyz="0.05 0.05 0.5" rpy="0 0 0"/>
-                <geometry>
-                    <box size="0.1 0.1 1.0"/>
-                </geometry>
-            </visual>
-            <collision>
-                <origin xyz="0.05 0.05 0.5" rpy="0 0 0"/>
-                <geometry>
-                    <box size="0.1 0.1 1.0"/>
-                </geometry>
-            </collision>
-            <inertial>
-                <mass value="1e2" />
-                <origin xyz="0.0 0.0 0.0" />
-                <inertia ixx = "0.000001" ixy = "0.000000" ixz = "0.000000"
-                         iyx = "0.000000" iyy = "0.000001" iyz = "0.000000"
-                         izx = "0.000000" izy = "0.000000" izz = "0.000001" />
-            </inertial>
-        </link>
-    </xacro:macro>
+<robot name="robotiq_85_gripper_sim_base" xmlns:xacro="http://www.ros.org/wiki/xacro">
+  <xacro:macro name="robotiq_85_gripper_sim_base" params="prefix">
+    <link name="${prefix}gripper_root_link">
+      <visual>
+        <origin xyz="0.05 0.05 0.5" rpy="0 0 0"/>
+        <geometry>
+          <box size="0.1 0.1 1.0"/>
+        </geometry>
+      </visual>
+      <collision>
+        <origin xyz="0.05 0.05 0.5" rpy="0 0 0"/>
+        <geometry>
+          <box size="0.1 0.1 1.0"/>
+        </geometry>
+      </collision>
+      <inertial>
+        <mass value="1e2" />
+        <origin xyz="0.0 0.0 0.0" />
+        <inertia ixx = "0.000001" ixy = "0.000000" ixz = "0.000000"
+             iyx = "0.000000" iyy = "0.000001" iyz = "0.000000"
+             izx = "0.000000" izy = "0.000000" izz = "0.000001" />
+      </inertial>
+    </link>
+  </xacro:macro>
 </robot>

Commit message: Improve grasping physics

File: robotiq_description/urdf/robotiq_85_gripper.transmission.xacro (robot description, xacro)
@@ -12,23 +12,17 @@
       </actuator>
     </transmission>
+    <!-- Mimic joints -->
     <gazebo>
-        <!-- loading plugin: mimic joints works in gazebo now -->
       <plugin filename="libgazebo_mimic_joint_plugin.so" name="${prefix}mimic_robotiq_85_1">
         <joint>${prefix}robotiq_85_left_knuckle_joint</joint>
         <mimicJoint>${prefix}robotiq_85_right_knuckle_joint</mimicJoint>
-        <!--multiplier>1.0</multiplier>
-        <offset>0.0</offset-->
       </plugin>
       <plugin filename="libgazebo_mimic_joint_plugin.so" name="${prefix}mimic_robotiq_85_2">
         <joint>${prefix}robotiq_85_left_knuckle_joint</joint>
         <mimicJoint>${prefix}robotiq_85_left_inner_knuckle_joint</mimicJoint>
-        <!--multiplier>1.0</multiplier>
-        <offset>0.0</offset-->
       </plugin>
       <plugin filename="libgazebo_mimic_joint_plugin.so" name="${prefix}mimic_robotiq_85_3">
         <joint>${prefix}robotiq_85_left_knuckle_joint</joint>
         <mimicJoint>${prefix}robotiq_85_right_inner_knuckle_joint</mimicJoint>
-        <!--multiplier>1.0</multiplier>
-        <offset>0.0</offset-->
       </plugin>
       <plugin filename="libgazebo_mimic_joint_plugin.so" name="${prefix}mimic_robotiq_85_4">

File: robotiq_description/urdf/robotiq_85_gripper.urdf.xacro (robot description, xacro)
@@ -32,5 +32,5 @@
       <axis xyz="0 0 1"/>
       <origin rpy="${pi} 0.0 0.0" xyz="0.05490451627 0.03060114443 0.0"/>
-      <limit lower="0.0" upper="0.804" velocity="2.0" effort="1000"/>
+      <limit lower="0.0" upper="0.80285" velocity="0.5" effort="1000"/>
     </joint>
     <joint name="${prefix}robotiq_85_right_knuckle_joint" type="continuous">
@@ -236,4 +236,19 @@
       </inertial>
     </link>
+    <!-- Improve grasping physics -->
+    <gazebo reference="${prefix}robotiq_85_left_finger_tip_link">
+      <kp>1000000.0</kp>
+      <kd>1.0</kd>
+      <mu1>1.0</mu1>
+      <mu2>1.0</mu2>
+      <minDepth>0.001</minDepth>
+    </gazebo>
+    <gazebo reference="${prefix}robotiq_85_right_finger_tip_link">
+      <kp>1000000.0</kp>
+      <kd>1.0</kd>
+      <mu1>1.0</mu1>
+      <mu2>1.0</mu2>
+      <minDepth>0.001</minDepth>
+    </gazebo>
     <xacro:robotiq_85_gripper_transmission prefix="${prefix}" />
   </xacro:macro>

Commit message: Rename main joint

File: robotiq_description/urdf/robotiq_85_gripper.transmission.xacro (robot description, xacro)
@@ -4,5 +4,5 @@
     <transmission name="${prefix}robotiq_85_left_knuckle_trans">
       <type>transmission_interface/SimpleTransmission</type>
-      <joint name="${prefix}robotiq_85_left_knuckle_joint">
+      <joint name="${prefix}finger_joint">
         <hardwareInterface>hardware_interface/PositionJointInterface</hardwareInterface>
       </joint>
@@ -15,17 +15,17 @@
     <gazebo>
       <plugin filename="libgazebo_mimic_joint_plugin.so" name="${prefix}mimic_robotiq_85_1">
-        <joint>${prefix}robotiq_85_left_knuckle_joint</joint>
+        <joint>${prefix}finger_joint</joint>
         <mimicJoint>${prefix}robotiq_85_right_knuckle_joint</mimicJoint>
       </plugin>
       <plugin filename="libgazebo_mimic_joint_plugin.so" name="${prefix}mimic_robotiq_85_2">
-        <joint>${prefix}robotiq_85_left_knuckle_joint</joint>
+        <joint>${prefix}finger_joint</joint>
         <mimicJoint>${prefix}robotiq_85_left_inner_knuckle_joint</mimicJoint>
       </plugin>
       <plugin filename="libgazebo_mimic_joint_plugin.so" name="${prefix}mimic_robotiq_85_3">
-        <joint>${prefix}robotiq_85_left_knuckle_joint</joint>
+        <joint>${prefix}finger_joint</joint>
         <mimicJoint>${prefix}robotiq_85_right_inner_knuckle_joint</mimicJoint>
       </plugin>
       <plugin filename="libgazebo_mimic_joint_plugin.so" name="${prefix}mimic_robotiq_85_4">
-        <joint>${prefix}robotiq_85_left_knuckle_joint</joint>
+        <joint>${prefix}finger_joint</joint>
         <mimicJoint>${prefix}robotiq_85_left_finger_tip_joint</mimicJoint>
         <multiplier>-1.0</multiplier>
@@ -33,5 +33,5 @@
       </plugin>
       <plugin filename="libgazebo_mimic_joint_plugin.so" name="${prefix}mimic_robotiq_85_5">
-        <joint>${prefix}robotiq_85_left_knuckle_joint</joint>
+        <joint>${prefix}finger_joint</joint>
         <mimicJoint>${prefix}robotiq_85_right_finger_tip_joint</mimicJoint>
         <multiplier>-1.0</multiplier>

File: robotiq_description/urdf/robotiq_85_gripper.urdf.xacro (robot description, xacro)
@@ -27,5 +27,5 @@
       </inertial>
     </link>
-    <joint name="${prefix}robotiq_85_left_knuckle_joint" type="revolute">
+    <joint name="${prefix}finger_joint" type="revolute">
       <parent link="${prefix}robotiq_85_base_link"/>
       <child link="${prefix}robotiq_85_left_knuckle_link"/>
@@ -40,5 +40,5 @@
       <origin rpy="0.0 0.0 0.0" xyz="0.05490451627 -0.03060114443 0.0"/>
       <limit lower="-3.14" upper="3.14" velocity="100.0" effort="1000"/>
-      <mimic joint="${prefix}robotiq_85_left_knuckle_joint"/>
+      <mimic joint="${prefix}finger_joint"/>
     </joint>
     <link name="${prefix}robotiq_85_left_knuckle_link">
@@ -134,5 +134,5 @@
       <origin xyz="0.06142 0.0127 0" rpy="${pi} 0.0 0.0" />
       <limit lower="-3.14" upper="3.14" velocity="100.0" effort="0.1"/>
-      <mimic joint="${prefix}robotiq_85_left_knuckle_joint" offset="0"/>
+      <mimic joint="${prefix}finger_joint" offset="0"/>
     </joint>
     <joint name="${prefix}robotiq_85_right_inner_knuckle_joint" type="continuous">
@@ -142,5 +142,5 @@
       <origin xyz="0.06142 -0.0127 0" rpy="0 0 0"/>
       <limit lower="-3.14" upper="3.14" velocity="100.0" effort="0.1"/>
-      <mimic joint="${prefix}robotiq_85_left_knuckle_joint" offset="0"/>
+      <mimic joint="${prefix}finger_joint" offset="0"/>
     </joint>
     <link name="${prefix}robotiq_85_left_inner_knuckle_link">
@@ -188,5 +188,5 @@
       <origin xyz="0.04303959807 -0.03759940821 0.0" rpy="0.0 0.0 0.0"/>
       <limit lower="-3.14" upper="3.14" velocity="100.0" effort="0.1"/>
-      <mimic joint="${prefix}robotiq_85_left_knuckle_joint" multiplier="-1"/>
+      <mimic joint="${prefix}finger_joint" multiplier="-1"/>
     </joint>
     <joint name="${prefix}robotiq_85_right_finger_tip_joint" type="continuous">
@@ -196,5 +196,5 @@
       <origin rpy="0.0 0.0 0.0" xyz="0.04303959807 -0.03759940821  0.0"/>
       <limit lower="-3.14" upper="3.14" velocity="100.0" effort="0.1"/>
-      <mimic joint="${prefix}robotiq_85_left_knuckle_joint" multiplier="-1"/>
+      <mimic joint="${prefix}finger_joint" multiplier="-1"/>
     </joint>
     <link name="${prefix}robotiq_85_left_finger_tip_link">
