Commit message: Fix hand-e mimic joint

File: robotiq_description/urdf/robotiq_hande_gripper.transmission.xacro (robot description, xacro)
@@ -2,5 +2,5 @@
 <robot xmlns:xacro="http://www.ros.org/wiki/xacro">
   <xacro:macro name="robotiq_hande_gripper_transmission" params="prefix">
-    <!-- <transmission name="${prefix}hande_left_finger_trans">
+    <transmission name="${prefix}hande_left_finger_trans">
       <type>transmission_interface/SimpleTransmission</type>
       <joint name="${prefix}hande_left_finger_joint">
@@ -10,6 +10,6 @@
         <mechanicalReduction>1</mechanicalReduction>
       </actuator>
-    </transmission> -->
-    <transmission name="${prefix}hande_right_finger_trans">
+    </transmission>
+    <!-- <transmission name="${prefix}hande_right_finger_trans">
       <type>transmission_interface/SimpleTransmission</type>
       <joint name="${prefix}hande_right_finger_joint">
@@ -19,10 +19,10 @@
         <mechanicalReduction>1</mechanicalReduction>
       </actuator>
-    </transmission>
+    </transmission> -->
     <!-- Mimic joints -->
     <gazebo>
       <plugin filename="libgazebo_mimic_joint_plugin.so" name="${prefix}mimic_robotiq_hande">
-        <joint>${prefix}hande_right_finger_joint</joint>
-        <mimicJoint>${prefix}hande_left_finger_joint</mimicJoint>
+        <joint>${prefix}hande_left_finger_joint</joint>
+        <mimicJoint>${prefix}hande_right_finger_joint</mimicJoint>
         <multiplier>1.0</multiplier>
         <offset>0.0</offset>

Commit message: fix hande

File: robotiq_description/urdf/robotiq_hande_gripper.transmission.xacro (robot description, xacro)
@@ -13,5 +13,5 @@
     <transmission name="${prefix}hande_right_finger_trans">
       <type>transmission_interface/SimpleTransmission</type>
-      <joint name="${prefix}hande_right_finger_joint">
+      <joint name="${prefix}finger_joint">
         <hardwareInterface>hardware_interface/PositionJointInterface</hardwareInterface>
       </joint>
@@ -23,5 +23,5 @@
     <gazebo>
       <plugin filename="libgazebo_mimic_joint_plugin.so" name="${prefix}mimic_robotiq_hande">
-        <joint>${prefix}hande_right_finger_joint</joint>
+        <joint>${prefix}finger_joint</joint>
         <mimicJoint>${prefix}hande_left_finger_joint</mimicJoint>
         <multiplier>1.0</multiplier>

File: robotiq_description/urdf/robotiq_hande_gripper.urdf.xacro (robot description, xacro)
@@ -4,5 +4,5 @@
   Author: Cristian Beltran
 -->
-  <xacro:include filename="$(find robotiq_description)/urdf/robotiq_hande_gripper.transmission.xacro" />
+  <xacro:include filename="$(find robotiq_description)/urdf/robotiq_arg2f_transmission.xacro" />
   <xacro:macro name="robotiq_hande_gripper" params="prefix parent *origin">
     <joint name="${prefix}robotiq_hande_base_joint" type="fixed">
@@ -86,5 +86,5 @@
       <material>Gazebo/Grey</material>
     </gazebo>
-    <joint name="${prefix}hande_left_finger_joint" type="prismatic">
+    <joint name="${prefix}finger_joint" type="prismatic">
       <origin rpy="0 0 0" xyz="0 0 0.099"/>
       <parent link="${prefix}hand_e_link"/>
@@ -99,5 +99,5 @@
       <axis xyz="1 0 0"/>
       <limit effort="130" lower="0" upper="0.025" velocity="0.15"/>
-      <mimic joint="${prefix}hande_left_finger_joint" multiplier="1" offset="0"/>
+      <mimic joint="${prefix}finger_joint" multiplier="1" offset="0"/>
     </joint>
       <!-- Improve grasping physics -->
@@ -116,5 +116,5 @@
         <minDepth>0.001</minDepth>
       </gazebo>
-    <xacro:robotiq_hande_gripper_transmission prefix="${prefix}" />
+    <xacro:robotiq_arg2f_transmission prefix="${prefix}"/>
   </xacro:macro>
 </robot>
